Commit message: Add support for exporting sites to URDF

File: test-fixtures/golden/3_DOF_ARM/expected.urdf (robot description, URDF)
Before this commit: robot 3_DOF_ARM - URDF, 4 links, 3 joints
Links:
- added link gripper
Joints:
- added joint gripper_joint: type fixed, parent effector_link, child gripper, origin xyz=0 0 0.0589644660940652 rpy=2.98632088395507E-16 0 -1.5707963267949
